File: esp32-dimmer/esp32_mc_dimmer.kicad_pcb (KiCad board)
At the start: 2 copper layers, 67 x 68 mm, 21 parts, among them J1 Conn_01x06, J2 Conn_01x04, J3 Conn_01x10, J4 Conn_01x02, J5 Conn_01x06, Q1 BUZ11, Q2 BUZ11, Q3 BUZ11, Q4 BUZ11, Q5 BUZ11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

Commit message: Add new psu module and improve power layout
Parts:
- added J6: Conn_01x06, Connector_PinHeader_2.54mm:PinHeader_1x06_P2.54mm_Vertical, F.Cu at (156.2, 121.9)
- C1: footprint Capacitor_THT:CP_Radial_D7.5mm_P2.50mm -> Capacitor_THT:CP_Radial_D10.0mm_P2.50mm_P5.00mm
- J2: footprint aOmat_osat:4pin_reg_con -> Voltage-regulator:4pin_reg_con
- J3: footprint aOmat_osat:Phoenix_SPTAF_1_10-5,0-EL -> Phoenix-connect:Phoenix_SPTAF_1_10-5,0-EL
- U1: footprint aOmat_osat:Doit_ESP32 -> esp32-doit-library:Doit_ESP32
- moved J2 13.4 mm to (134.0, 102.9)
- moved C1 2.22 mm to (128.9, 80.6), turned to 270 degrees
- moved R1 0.89 mm to (135.9, 76.5)
- moved J5 0.52 mm to (156.2, 125.5)
Routing:
- net +3V3: track 124.0 -> 112.2 mm
- net +12C: track 37.2 -> 46.5 mm
- net RX: track 26.5 -> 31.3 mm
- net TX: track 26.0 -> 30.7 mm
- net +12V: track 166.9 -> 166.0 mm
Other:
- board text added: "12-24V"
- board text added: "6-Channel LED dimmer v2 Doit ESP32, or ESP32-WROOM-32D Mikko Tervala, 19.2020"
- board text removed: "+12V"
- board text removed: "6-Channel LED dimmer Doit ESP32, or ESP32-WROOM-32D Mikko Tervala, 8.2019"

Commit message: Change resistor to lower inrush
Parts:
- U2: value ESP32-WROOM-32D -> ESP32-WROOM-32
Other:
- board text added: "R1 5Ω Or R2 5Ω Or JP1"
- board text removed: "R1 1Ω Or R2 1Ω Or JP1"
